File: kicad-and-mfg/keyboard/kicad/bitseithr-keyboard.kicad_sch (KiCad schematic)
At the start: 74 parts, among them P1 KEYB CONN 1

Commit message: changeed path, migrated to kicad 10
Parts:
- removed P1: KEYB CONN 1, EasyEDA_Lib:IDC-TH_20P-L33.0-W13.8-H-M-R2-C10-P2.54-S2.54-TR, symbol EasyEDA_Lib:IDC Box 2X10 2.54MM
- added P2: KEYB CONN 1, EasyEDA_Lib:IDC-TH_20P-L33.0-W13.8-H-M-R2-C10-P2.54-S2.54-TR, symbol EasyEDA_Lib:IDC Box 2X10 2.54MM
- D10, D11, D12, D13, D14, D15, D16, D17, D18, D19, D2, D20, D21, D22, D23, D24, D25, D26, D27, D28, D29, D3, D30, D31, D32, D33, D34, D35, D36, D4, D5, D6, D7, D8, D9: footprint Diode_THT:D_DO-35_SOD27_P7.62mm_Horizontal -> EasyEDA_Lib:SOD-523_L1.2-W0.8-LS1.6-RD-1
- MX1, MX10, MX11, MX12, MX13, MX14, MX16, MX17, MX18, MX19, MX2, MX20, MX21, MX22, MX23, MX24, MX25, MX26, MX27, MX28, MX29, MX3, MX30, MX31, MX32, MX33, MX34, MX35, MX4, MX5, MX6, MX7, MX8, MX9: footprint cholm-footprints:MXOnly-1U-NoLED -> clholm-kicad-library:MX-Hotswap-1U
- MX15: footprint cholm-footprints:MXOnly-2.25U-NoLED -> clholm-kicad-library:MX-Hotswap-2.25U
- R16: footprint (none) -> EasyEDA_Lib:R0805
Connections:
- net +9V: now also P2.2
- net COL0: now also P2.3
- net COL1: now also P2.5
- net COL2: now also P2.7
- net COL3: now also P2.9
- net COL4: now also P2.11
- net COL5: now also P2.13
- net COL6: now also P2.15
- net COL7: now also P2.17
- net COL8: now also MX34.1 (COL), MX35.1 (COL), P2.19
- net GND: now also P2.4
- net ROW0: now also P2.10
- net ROW1: now also P2.12
- net ROW2: now also P2.14
- net ROW3: now also P2.16
- net ROW4: now also P2.18
- net ROW5: now also P2.20
Other:
- moved on the sheet: D10, D11, D12, D13, D14, D15, D16, D17, D18, D19, D2, D20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
